Commit message: use simple geometry collision

File: legged_rl_description/urdf/biped.urdf (robot description, URDF)
Before this commit: robot biped, 20 links, 19 joints
Links:
- link abad_L_Link: geometry collision cylinder length=0.15 radius=0.05; visual mesh filename=package://legged_rl_description/meshes/biped/abad_left_link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
- link abad_R_Link: geometry collision cylinder length=0.15 radius=0.05; visual mesh filename=package://legged_rl_description/meshes/biped/abad_right_lin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
- link base: geometry collision box size=0.2 0.3 0.15; visual mesh filename=package://legged_rl_description/meshes/biped/base_link.STL
- link foot_L_Link: geometry collision sphere radius=0.035; visual mesh filename=package://legged_rl_description/meshes/biped/foot_left_link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
- link foot_R_Link: geometry collision sphere radius=0.035; visual mesh filename=package://legged_rl_description/meshes/biped/foot_right_lin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
- link hip_L_Link: geometry collision cylinder length=0.22 radius=0.035; visual mesh filename=package://legged_rl_description/meshes/biped/hip_left_link.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
- link hip_R_Link: geometry collision cylinder length=0.22 radius=0.035; visual mesh filename=package://legged_rl_description/meshes/biped/hip_right_link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
- link knee_L_Link: geometry collision cylinder length=0.26 radius=0.015; visual mesh filename=package://legged_rl_description/meshes/biped/knee_left_link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
- link knee_R_Link: geometry collision cylinder length=0.26 radius=0.015; visual mesh filename=package://legged_rl_description/meshes/biped/knee_right_lin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

Commit message: tmp commit, this policy is not fine

File: legged_rl_description/urdf/biped.urdf (robot description, URDF)
Before this commit: robot biped, 20 links, 19 joints
Links:
- link foot_L_Link: geometry collision sphere radius=0.04; visual mesh filename=package://legged_rl_description/meshes/biped/foot_left_link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
- link foot_R_Link: geometry collision sphere radius=0.04; visual mesh filename=package://legged_rl_description/meshes/biped/foot_right_lin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
Joints:
- joint abad_L_Joint: limit lower=-0.69813 upper=1.39626 effort=20 velocity=52.4 -> lower=-0.383972435 upper=0.785398163 effort=80.0 velocity=20.0
- joint abad_R_Joint: axis -1 0 0 -> 1 0 0; limit lower=-0.69813 upper=1.39626 effort=30 velocity=52.4 -> lower=-0.785398163 upper=0.383972435 effort=80.0 velocity=20.0
- joint hip_L_Joint: axis 0 -1 0 -> 0 1 0; limit lower=-1.012 upper=1.012 effort=30 velocity=52.4 -> lower=-1.047197551 upper=1.483529864 effort=80.0 velocity=20.0
- joint hip_R_Joint: limit lower=-1.012 upper=1.012 effort=30 velocity=52.4 -> lower=-1.483529864 upper=1.047197551 effort=80.0 velocity=20.0
- joint knee_L_Joint: limit lower=-1.04719 upper=1.39626 effort=30 velocity=52.4 -> lower=-1.012290966 upper=1.256637061 effort=80 velocity=20
- joint knee_R_Joint: limit lower=-1.39626 upper=1.04719 effort=30 velocity=52.4 -> lower=-1.256637061 upper=1.012290966 effort=80 velocity=20
